File: Hardware/Eagle_Design/CAN_Wake_Up_2.brd (EAGLE design)
At the start: 65 x 32 mm, 39 parts, among them IC1 STM32F10XCXT6, IC4 LM1117MP-5.0, IC5 LM1117MP-3.3, Q1 8MHz

Commit message: Fixed ignores again
Parts:
- removed POWER: (no value), pinhead:1X02
- added GND, KL30: (no value), pinhead:1X01
- moved H1 11.4 mm to (14.4, 27.9)
- moved H2 11.4 mm to (14.4, 3.81)
- moved C8 8.52 mm to (5.08, 7.62), turned to 90 degrees
- moved C5 8.03 mm to (5.08, 25.4)
- moved C6 1.80 mm to (10.2, 29.2), turned to 180 degrees
- moved C13 1.27 mm to (17.8, 11.4)
- moved C14 1.27 mm to (17.8, 21.6)
- moved C15 1.27 mm to (22.9, 21.6)
- moved C7 1.27 mm to (10.2, 3.81), turned to 180 degrees
- moved IC5 1.27 mm to (11.4, 22.9)
- moved H4 0.11 mm to (49.8, 22.9)
Connections:
- new net CAN__TX_MCU: IC1.33
- net CAN_TX_MCU: no longer IC1.33
- net GND: now also DEBUG.4, GND.1; no longer POWER.2
- net KL30: now also KL30.1; no longer POWER.1
- net VCC_3V3: now also DEBUG.1
Routing:
- net LED_MCU_PWR: track 36.7 -> 52.8 mm, vias 2 -> 0
- net N$8: track 31.9 -> 19.2 mm, vias 0 -> 2
- net KL30: track 38.0 -> 26.8 mm, vias 1 -> 0
- net CAN_TX_MCU: track 8.68 -> 0.00 mm
- net DBG_SWDIO: track 38.8 -> 30.8 mm, vias 1 -> 0
- net LED_MCU_CAN: track 26.1 -> 34.0 mm
- net N$1: track 19.6 -> 12.3 mm, vias 0 -> 2
- net VCC_3V3: track 96.6 -> 90.7 mm, vias 4 -> 3
- net CAN_RX_MCU: track 10.7 -> 16.5 mm
- net N$9: track 15.7 -> 10.9 mm
- net N$6: track 17.4 -> 12.9 mm
- net USART1_TX: track 29.1 -> 25.4 mm
- net DBG_SWCLK: track 21.0 -> 17.4 mm, vias 2 -> 0
- net USART_1_RX: track 20.5 -> 22.5 mm
- net VCC_5V: track 54.2 -> 53.2 mm
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Other:
- board text removed: "GND"
- board text removed: "KL30"
- board text removed: "RX"
- board text removed: "TX"
