File: Hardware/Eagle_Design/CAN_Wake_Up.brd (EAGLE design)
At the start: 65 x 32 mm, 39 parts, among them IC1 STM32F10XCXT6, IC4 LM1117MP-5.0, IC5 LM1117MP-3.3, Q1 8MHz

Commit message: Latest hardware revision: rev2
Parts:
- DEBUG: device pinhead:1X04 -> pinhead:1X05
- moved SERIAL 24.3 mm to (20.3, 27.9)
- moved S1 14.0 mm to (21.6, 3.50)
- moved R1 13.1 mm to (33.0, 16.5), flipped to the bottom
- moved R8 12.5 mm to (12.7, 16.5), flipped to the bottom
- moved DEBUG 8.89 mm to (31.8, 27.9)
- moved R6 8.52 mm to (27.9, 24.1), flipped to the bottom, turned to 0 degrees
- moved C10 8.13 mm to (41.9, 22.4), flipped to the top
- moved C1 7.62 mm to (40.1, 16.0)
- moved C12 6.72 mm to (41.9, 9.40), turned to 270 degrees
- moved C7 6.35 mm to (8.89, 10.2), flipped to the bottom, turned to 90 degrees
- moved C8 6.35 mm to (12.7, 10.2), flipped to the bottom, turned to 90 degrees
- moved C3 5.68 mm to (31.8, 5.08), flipped to the top, turned to 270 degrees
- moved C4 5.08 mm to (35.6, 5.08), flipped to the top, turned to 270 degrees
- moved R7 4.58 mm to (34.3, 24.1), flipped to the bottom, turned to 0 degrees
- moved C5 3.81 mm to (12.7, 24.1), flipped to the bottom
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Connections:
- net GND: now also DEBUG.4
- net N$9: now also DEBUG.5
- net VCC_3V3: now also DEBUG.1
Routing:
- net LED_MCU_PWR: track 36.7 -> 54.9 mm, vias 2 -> 0
- net N$1: track 19.6 -> 3.56 mm, vias 0 -> 1
- net N$9: track 15.7 -> 30.0 mm
- net DBG_SWDIO: track 38.8 -> 24.8 mm
- net USART_1_RX: track 20.5 -> 33.0 mm
- net N$7: track 12.3 -> 22.4 mm
- net N$8: track 31.9 -> 24.5 mm, vias 0 -> 1
- net USART1_TX: track 29.1 -> 35.7 mm
- net CAN_S_MCU: track 17.8 -> 23.4 mm
- net DBG_SWCLK: track 21.0 -> 15.6 mm, vias 2 -> 0
- net N$6: track 17.4 -> 12.6 mm
- net KL30: track 38.0 -> 42.2 mm, vias 1 -> 0
- net VCC_5V: track 54.2 -> 50.2 mm, vias 2 -> 1
- net LED_MCU_CAN: track 26.1 -> 22.7 mm
- net N$5: track 13.6 -> 10.3 mm
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Other:
- board text added: "3V3"
- board text added: "CANWakeUp v2 Jonas Heim 03.2019"
- board text added: "RST"
- board text added: "SWCLK"
- board text added: "SWDIO"
- board text removed: "CANWakeUp v2 J.Heim 03.2019"
